Commit message: Localization, navigation and new sensors

File: waiter_robot_description/urdf/lidar.xacro (robot description, xacro)
@@ -47,5 +47,5 @@
         <sensor name="laser" type="ray">
             <pose> 0 0 0 0 0 0 </pose>
-            <visualize>true</visualize>
+            <visualize>false</visualize>
             <update_rate>10</update_rate>
             <ray>

File: waiter_robot_description/urdf/waiter_robot.xacro (robot description, xacro)
@@ -5,3 +5,4 @@
     <xacro:include filename="lidar.xacro" />
     <xacro:include filename="camera.xacro" />
+    <xacro:include filename="bumper.xacro" />
 </robot>

File: waiter_robot_description/urdf/waiter_robot_core.xacro (robot description, xacro)
@@ -247,17 +247,4 @@
     <origin xyz="0 0 0.3"/>
   </joint>
-  <!-- <link name="box">
-    <visual>
-      <geometry>
-        <box size="0.08 0.08 0.08"/>
-      </geometry>
-      <material name="white"/>
-    </visual>
-  </link>
-  <joint name="tobox" type="fixed">
-    <parent link="head"/>
-    <child link="box"/>
-    <origin xyz="0.1814 0 0.1414"/>
-  </joint> -->
 <link name="tray_pole">
   <visual>
