Commit message: Update master launch file to integrate waiter robot, adjust Gazebo launch parameters, and modify robot state publisher. Change base frame ID in navigation parameters and fix bumper collision reference in URDF.

File: waiter_robot_description/urdf/bumper.xacro (robot description, xacro)
@@ -27,5 +27,5 @@
     <update_rate>10</update_rate>
     <contact>
-      <collision>bumper_link_collision</collision>
+      <collision>bumper_collision</collision>
     </contact>
     <plugin name="bumper_plugin" filename="libgazebo_ros_bumper.so">

Commit message: April Tag detection package

File: waiter_robot_description/urdf/bumper.xacro (robot description, xacro)
@@ -36,5 +36,5 @@
       <frameName>bumper_link</frameName>
     </plugin>
-  </sensor>
-</gazebo>
+    </sensor>
+    </gazebo>
 </robot>

File: waiter_robot_description/urdf/camera.xacro (robot description, xacro)
@@ -4,5 +4,5 @@
         <parent link="head"/>
         <child link="camera_link"/>
-        <origin xyz="0 0 0.22" rpy="0 0 0"/>
+        <origin xyz="0 0 0.22" rpy="0 0.15 0"/>
     </joint>
     <link name="camera_link">
